Commit message: Imported upstream version '4.0.0' of 'upstream'

File: urdf/inc/ur_common.xacro (robot description, xacro)
@@ -21,5 +21,10 @@
   </xacro:macro>
   <xacro:macro name="get_visual_params" params="name:=^ type:=^" >
-    <xacro:property name="visual_params" value="${sec_mesh_files[name][type]}" scope="parent"/>
+    <xacro:if value="${type in sec_mesh_files[name]}">
+      <xacro:property name="visual_params" value="${sec_mesh_files[name][type]}" scope="parent"/>
+    </xacro:if>
+    <xacro:unless value="${type in sec_mesh_files[name]}">
+      <xacro:property name="visual_params" value="" scope="parent"/>
+    </xacro:unless>
   </xacro:macro>
   <!-- Simplification of getting meshes. Available types can be seen in the visual_parameters.yaml (At the time of writing: visual, collision) -->
@@ -46,5 +51,4 @@
     <!-- Extract subsections from yaml dictionaries -->
     <xacro:property name="sec_limits" value="${config_joint_limit_parameters['joint_limits']}"/>
-    <xacro:property name="sec_offsets" value="${config_physical_parameters['offsets']}"/>
     <xacro:property name="sec_inertia_parameters" value="${config_physical_parameters['inertia_parameters']}" />
     <xacro:property name="sec_mesh_files" value="${config_visual_parameters['mesh_files']}" scope="parent"/>
@@ -118,7 +122,4 @@
     <xacro:property name="wrist_3_pitch" value="${sec_kinematics['wrist_3']['pitch']}" scope="parent"/>
     <xacro:property name="wrist_3_yaw" value="${sec_kinematics['wrist_3']['yaw']}" scope="parent"/>
-    <!-- OFFSETS -->
-    <xacro:property name="shoulder_offset" value="${sec_offsets['shoulder_offset']}" scope="parent"/>
-    <xacro:property name="elbow_offset" value="${sec_offsets['elbow_offset']}" scope="parent"/>
     <!-- INERTIA PARAMETERS -->
     <!-- mass -->
@@ -203,10 +204,4 @@
     <xacro:property name="wrist_3_inertia_iyz" value="${prop_wrist_3_inertia['iyz']}" scope="parent"/>
     <xacro:property name="wrist_3_inertia_izz" value="${prop_wrist_3_inertia['izz']}" scope="parent"/>
-    <!-- cylinder radius -->
-    <xacro:property name="shoulder_radius" value="${sec_inertia_parameters['shoulder_radius']}" scope="parent"/>
-    <xacro:property name="upper_arm_radius" value="${sec_inertia_parameters['upper_arm_radius']}" scope="parent"/>
-    <xacro:property name="elbow_radius" value="${sec_inertia_parameters['elbow_radius']}" scope="parent"/>
-    <xacro:property name="forearm_radius" value="${sec_inertia_parameters['forearm_radius']}" scope="parent"/>
-    <xacro:property name="wrist_radius" value="${sec_inertia_parameters['wrist_radius']}" scope="parent"/>
     <!--KINEMATICS HASH-->
     <xacro:property name="kinematics_hash" value="${sec_kinematics['hash']}" scope="parent"/>

File: urdf/ur.urdf.xacro (robot description, xacro)
@@ -5,5 +5,5 @@
    <!-- import main macro -->
    <xacro:include filename="$(find ur_description)/urdf/ur_macro.xacro"/>
-   <!-- possible 'ur_type' values: ur3, ur3e, ur5, ur5e, ur10, ur10e, ur16e, ur20, ur30 -->
+   <!-- possible 'ur_type' values: ur3, ur3e, ur5, ur5e, ur7e, ur10, ur10e, ur12e, ur16e, ur15, ur20, ur30 -->
    <!-- the default value should raise an error in case this was called without defining the type -->
    <xacro:arg name="ur_type" default="ur5x"/>

File: urdf/ur_macro.xacro (robot description, xacro)
@@ -65,8 +65,17 @@
       force_abs_paths="${force_abs_paths}"/>
     <!-- links -  main serial chain -->
+    <!-- base_link serves as the root of the robot's kinematic tree. It follows REP-103
+        conventions (i.e., X+ forward, Y+ left, Z+ up).
+        Since some kinematic solvers forbid having inertia values attached to a root link, we've
+        added the base_link_inertia link that carries the visual, collision and inertia
+        information.
+    -->
     <link name="${tf_prefix}base_link"/>
     <link name="${tf_prefix}base_link_inertia">
-      <visual>
-        <origin xyz="0 0 0" rpy="0 0 ${pi}"/>
+      <xacro:get_visual_params name="base" type="mesh_offset"/>
+      <visual>
+        <origin
+         xyz="${visual_params['x']} ${visual_params['y']} ${visual_params['z']}"
+         rpy="${visual_params['roll']} ${visual_params['pitch']} ${visual_params['yaw']}"/>
         <geometry>
           <xacro:get_mesh name="base" type="visual"/>
@@ -74,5 +83,7 @@
       </visual>
       <collision>
-        <origin xyz="0 0 0" rpy="0 0 ${pi}"/>
+        <origin
+         xyz="${visual_params['x']} ${visual_params['y']} ${visual_params['z']}"
+         rpy="${visual_params['roll']} ${visual_params['pitch']} ${visual_params['yaw']}"/>
         <geometry>
           <xacro:get_mesh name="base" type="collision"/>
@@ -84,6 +95,9 @@
     </link>
     <link name="${tf_prefix}shoulder_link">
-      <visual>
-        <origin xyz="0 0 0" rpy="0 0 ${pi}"/>
+      <xacro:get_visual_params name="shoulder" type="mesh_offset"/>
+      <visual>
+        <origin
+         xyz="${visual_params['x']} ${visual_params['y']} ${visual_params['z']}"
+         rpy="${visual_params['roll']} ${visual_params['pitch']} ${visual_params['yaw']}"/>
         <geometry>
           <xacro:get_mesh name="shoulder" type="visual"/>
@@ -91,5 +105,7 @@
       </visual>
       <collision>
-        <origin xyz="0 0 0" rpy="0 0 ${pi}"/>
+        <origin
+         xyz="${visual_params['x']} ${visual_params['y']} ${visual_params['z']}"
+         rpy="${visual_params['roll']} ${visual_params['pitch']} ${visual_params['yaw']}"/>
         <geometry>
           <xacro:get_mesh name="shoulder" type="collision"/>
@@ -109,6 +125,9 @@
       </inertial>    </link>
     <link name="${tf_prefix}upper_arm_link">
-      <visual>
-        <origin xyz="0 0 ${shoulder_offset}" rpy="${pi/2} 0 ${-pi/2}"/>
+      <xacro:get_visual_params name="upper_arm" type="mesh_offset"/>
+      <visual>
+        <origin
+         xyz="${visual_params['x']} ${visual_params['y']} ${visual_params['z']}"
+         rpy="${visual_params['roll']} ${visual_params['pitch']} ${visual_params['yaw']}"/>
         <geometry>
           <xacro:get_mesh name="upper_arm" type="visual"/>
@@ -116,5 +135,7 @@
       </visual>
       <collision>
-        <origin xyz="0 0 ${shoulder_offset}" rpy="${pi/2} 0 ${-pi/2}"/>
+        <origin
+         xyz="${visual_params['x']} ${visual_params['y']} ${visual_params['z']}"
+         rpy="${visual_params['roll']} ${visual_params['pitch']} ${visual_params['yaw']}"/>
         <geometry>
           <xacro:get_mesh name="upper_arm" type="collision"/>
@@ -135,6 +156,9 @@
     </link>
     <link name="${tf_prefix}forearm_link">
-      <visual>
-        <origin xyz="0 0 ${elbow_offset}" rpy="${pi/2} 0 ${-pi/2}"/>
+      <xacro:get_visual_params name="forearm" type="mesh_offset"/>
+      <visual>
+        <origin
+         xyz="${visual_params['x']} ${visual_params['y']} ${visual_params['z']}"
+         rpy="${visual_params['roll']} ${visual_params['pitch']} ${visual_params['yaw']}"/>
         <geometry>
           <xacro:get_mesh name="forearm" type="visual"/>
@@ -142,5 +166,7 @@
       </visual>
       <collision>
-        <origin xyz="0 0 ${elbow_offset}" rpy="${pi/2} 0 ${-pi/2}"/>
+        <origin
+         xyz="${visual_params['x']} ${visual_params['y']} ${visual_params['z']}"
+         rpy="${visual_params['roll']} ${visual_params['pitch']} ${visual_params['yaw']}"/>
         <geometry>
           <xacro:get_mesh name="forearm" type="collision"/>
@@ -161,7 +187,9 @@
     </link>
     <link name="${tf_prefix}wrist_1_link">
-	  <xacro:get_visual_params name="wrist_1" type="visual_offset"/>
-      <visual>
-      	<origin xyz="0 0 ${visual_params}" rpy="${pi/2} 0 0"/>
+      <xacro:get_visual_params name="wrist_1" type="mesh_offset"/>
+      <visual>
+        <origin
+         xyz="${visual_params['x']} ${visual_params['y']} ${visual_params['z']}"
+         rpy="${visual_params['roll']} ${visual_params['pitch']} ${visual_params['yaw']}"/>
         <geometry>
           <xacro:get_mesh name="wrist_1" type="visual"/>
@@ -169,5 +197,7 @@
       </visual>
       <collision>
-        <origin xyz="0 0 ${visual_params}" rpy="${pi/2} 0 0"/>
+        <origin
+         xyz="${visual_params['x']} ${visual_params['y']} ${visual_params['z']}"
+         rpy="${visual_params['roll']} ${visual_params['pitch']} ${visual_params['yaw']}"/>
         <geometry>
           <xacro:get_mesh name="wrist_1" type="collision"/>
@@ -188,7 +218,9 @@
     </link>
     <link name="${tf_prefix}wrist_2_link">
-	  <xacro:get_visual_params name="wrist_2" type="visual_offset"/>
-      <visual>
-        <origin xyz="0 0 ${visual_params}" rpy="0 0 0"/>
+      <xacro:get_visual_params name="wrist_2" type="mesh_offset"/>
+      <visual>
+        <origin
+         xyz="${visual_params['x']} ${visual_params['y']} ${visual_params['z']}"
+         rpy="${visual_params['roll']} ${visual_params['pitch']} ${visual_params['yaw']}"/>
         <geometry>
           <xacro:get_mesh name="wrist_2" type="visual"/>
@@ -196,5 +228,7 @@
       </visual>
       <collision>
-        <origin xyz="0 0 ${visual_params}" rpy="0 0 0"/>
+        <origin
+         xyz="${visual_params['x']} ${visual_params['y']} ${visual_params['z']}"
+         rpy="${visual_params['roll']} ${visual_params['pitch']} ${visual_params['yaw']}"/>
         <geometry>
           <xacro:get_mesh name="wrist_2" type="collision"/>
@@ -215,7 +249,9 @@
     </link>
     <link name="${tf_prefix}wrist_3_link">
-	  <xacro:get_visual_params name="wrist_3" type="visual_offset"/>
-      <visual>
-        <origin xyz="0 0 ${visual_params}" rpy="${pi/2} 0 0"/>
+      <xacro:get_visual_params name="wrist_3" type="mesh_offset"/>
+      <visual>
+        <origin
+         xyz="${visual_params['x']} ${visual_params['y']} ${visual_params['z']}"
+         rpy="${visual_params['roll']} ${visual_params['pitch']} ${visual_params['yaw']}"/>
         <geometry>
           <xacro:get_mesh name="wrist_3" type="visual"/>
@@ -223,5 +259,7 @@
       </visual>
       <collision>
-        <origin xyz="0 0 ${visual_params}" rpy="${pi/2} 0 0"/>
+        <origin
+         xyz="${visual_params['x']} ${visual_params['y']} ${visual_params['z']}"
+         rpy="${visual_params['roll']} ${visual_params['pitch']} ${visual_params['yaw']}"/>
         <geometry>
           <xacro:get_mesh name="wrist_3" type="collision"/>

File: urdf/ur_mocked.urdf.xacro (robot description, xacro)
@@ -6,5 +6,5 @@
   <xacro:include filename="$(find ur_description)/urdf/ur_macro.xacro"/>
   <xacro:include filename="$(find ur_description)/urdf/ros2_control_mock_hardware.xacro" />
-  <!-- possible 'ur_type' values: ur3, ur3e, ur5, ur5e, ur10, ur10e, ur16e, ur20, ur30 -->
+  <!-- possible 'ur_type' values: ur3, ur3e, ur5, ur5e, ur7e, ur10, ur10e, ur12e, ur16e, ur15, ur20, ur30 -->
   <!-- the default value should raise an error in case this was called without defining the type -->
   <xacro:arg name="ur_type" default="ur5x"/>
